File: Hardware/Redbox_Explorer_Cartridge.kicad_sch (KiCad schematic)
At the start: 51 parts, among them Q1 BS170, Q10 BS170, Q11 BS170, Q12 BS170, Q13 BS170, Q14 BS170, Q15 BS170, Q2 BS170, Q3 BS170, Q4 BS170, Q5 BS170, Q6 BS170, Q7 BS170, Q8 BS170, Q9 BS170, U1 MCP3008

Commit message: Project structure: hardware
Other:
- note added: "Red[box] Explorer Cartridge"
- note added: "Rev. 1.1, early 2025"
- note removed: "EDGEBERRY CARTRIDGE"
- note removed: "Edge Explorer Rev. 1.1, early 2025"
Changed lines of the file:
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@@
 		)
 	)
-	(text "Edge Explorer Rev. 1.1, early 2025"
+	(text "Rev. 1.1, early 2025"
 		(exclude_from_sim no)
 		(at 179.07 175.26 0)
@@
 		)
 	)
-	(text "EDGEBERRY CARTRIDGE"
+	(text "Red[box] Explorer Cartridge"
 		(exclude_from_sim no)
 		(at 178.816 173.99 0)
